Commit message: More bullshit

File: src/rhex_description/urdf/macros.xacro (robot description, xacro)
@@ -30,5 +30,5 @@
       <axis xyz="1 0 0"/>
       <limit effort="30" velocity="4"/>
-      <dynamics damping="0.1" friction="0.1"/>\
+      <dynamics damping="1.0" friction="1.0"/>\
     </joint>
   </xacro:macro>

File: src/rhex_description/urdf/rhex.control.xacro (robot description, xacro)
@@ -7,30 +7,30 @@
       </hardware>
       <joint name="front_left_leg_joint">
-        <command_interface name="effort"/>
+        <command_interface name="position"/>
         <state_interface name="position"/>
         <state_interface name="velocity"/>
       </joint>
       <joint name="centre_left_leg_joint">
-        <command_interface name="effort"/>
+        <command_interface name="position"/>
         <state_interface name="position"/>
         <state_interface name="velocity"/>
       </joint>
       <joint name="back_left_leg_joint">
-        <command_interface name="effort"/>
+        <command_interface name="position"/>
         <state_interface name="position"/>
         <state_interface name="velocity"/>
       </joint>
       <joint name="front_right_leg_joint">
-        <command_interface name="effort"/>
+        <command_interface name="position"/>
         <state_interface name="position"/>
         <state_interface name="velocity"/>
       </joint>
       <joint name="centre_right_leg_joint">
-        <command_interface name="effort"/>
+        <command_interface name="position"/>
         <state_interface name="position"/>
         <state_interface name="velocity"/>
       </joint>
       <joint name="back_right_leg_joint">
-        <command_interface name="effort"/>
+        <command_interface name="position"/>
         <state_interface name="position"/>
         <state_interface name="velocity"/>

Commit message: balls

File: src/rhex_description/urdf/macros.xacro (robot description, xacro)
@@ -1,4 +1,4 @@
 <robot xmlns:xacro="http://ros.org/wiki/xacro">
-  <xacro:macro name="leg_link" params="name mesh">
+  <xacro:macro name="leg_link" params="name mesh xyz">
     <link name="${name}">
       <visual>
@@ -14,7 +14,7 @@
       </collision>
       <inertial>
-        <mass value="0.024174555469373752"/>
-        <origin xyz="0 0 0"/>
-        <inertia ixx="0.00011" ixy="0.0" ixz="0.0" iyy="0.00013" iyz="-0.0" izz="2.1e-05"/>
+        <mass value="0.064"/>
+        <origin xyz="${xyz}"/>
+        <inertia ixx="0.000143" ixy="-0.000000832" ixz="0.00000113" iyy="0.000114" iyz="0.0000159" izz="0.0000389"/>
       </inertial>
     </link>

File: src/rhex_description/urdf/rhex.control.xacro (robot description, xacro)
@@ -1,40 +1,21 @@
 <?xml version="1.0"?>
 <robot xmlns:xacro="http://www.ros.org/wiki/xacro">
-  <xacro:macro name="rhex_control" params="">
-    <ros2_control name="RHexHardware" type="system">
-      <hardware>
-        <plugin>gazebo_ros2_control/GazeboSystem</plugin>
-      </hardware>
-      <joint name="front_left_leg_joint">
-        <command_interface name="position"/>
-        <state_interface name="position"/>
-        <state_interface name="velocity"/>
-      </joint>
-      <joint name="centre_left_leg_joint">
-        <command_interface name="position"/>
-        <state_interface name="position"/>
-        <state_interface name="velocity"/>
-      </joint>
-      <joint name="back_left_leg_joint">
-        <command_interface name="position"/>
-        <state_interface name="position"/>
-        <state_interface name="velocity"/>
-      </joint>
-      <joint name="front_right_leg_joint">
-        <command_interface name="position"/>
-        <state_interface name="position"/>
-        <state_interface name="velocity"/>
-      </joint>
-      <joint name="centre_right_leg_joint">
-        <command_interface name="position"/>
-        <state_interface name="position"/>
-        <state_interface name="velocity"/>
-      </joint>
-      <joint name="back_right_leg_joint">
-        <command_interface name="position"/>
-        <state_interface name="position"/>
-        <state_interface name="velocity"/>
-      </joint>
-    </ros2_control>
+  <xacro:macro name="rhex_control" params="use_sim:=false">
+    <xacro:if value="${use_sim}">
+      <ros2_control name="RHexHardware" type="system">
+        <hardware>
+          <plugin>gazebo_ros2_control/GazeboSystem</plugin>
+        </hardware>
+        <xacro:include filename="$(find rhex_description)/urdf/joints_interfaces.xacro"/>
+      </ros2_control>
+    </xacro:if>
+    <xacro:unless value="${use_sim}">
+      <ros2_control name="GigaHardware" type="system">
+        <hardware>
+          <plugin>giga_hw_interface/GigaHardwareInterface</plugin>
+        </hardware>
+        <xacro:include filename="$(find rhex_description)/urdf/joints_interfaces.xacro"/>
+      </ros2_control>
+    </xacro:unless>
   </xacro:macro>
 </robot>

File: src/rhex_description/urdf/rhex.xacro (robot description, xacro)
@@ -24,19 +24,109 @@
     </collision>
     <inertial>
-      <mass value="3.703374358474152"/>
-      <origin xyz="0 0 0"/>
-      <inertia ixx="0.020087" ixy="-0.0" ixz="-0.0" iyy="0.090417" iyz="0.0" izz="0.108396"/>
+      <mass value="1.5"/>
+      <origin xyz="0 0 0.05"/>
+      <inertia ixx="2.222e-2" ixy="4.654e-6" ixz="1.02836e-5" iyy="1.129e-2" iyz="4.82214e-5" izz="2.96e-2"/>
     </inertial>
   </link>
+  <link name="lidar_link">
+  <visual>
+    <origin xyz="0 0 0" rpy="0 0 0"/>
+    <geometry>
+      <mesh filename="$(find rhex_description)/meshes/lidar.stl" scale="1 1 1"/>
+    </geometry>
+    <material name="gray"/>
+  </visual>
+  <inertial>
+    <mass value="0.073"/>
+    <origin xyz="0 0 0"/>
+    <inertia ixx="0.0000615" ixy="0.000000596" ixz="0.00000038" iyy="3.17e-5" iyz="-6.53e-6" izz="7.2e-5"/>
+  </inertial>
+</link>
+<joint name="lidar_mount" type="fixed">
+  <parent link="base_link"/>
+  <child link="lidar_link"/>
+  <origin xyz="0 -0.045 0.1" rpy="0 0 0"/>
+</joint>
+<link name="stereo_camera_link">
+  <visual>
+    <origin xyz="0 0 0" rpy="0 0 0"/>
+    <geometry>
+      <mesh filename="$(find rhex_description)/meshes/stereo_camera.stl" scale="1 1 1"/>
+    </geometry>
+    <material name="gray"/>
+  </visual>
+  <inertial>
+    <mass value="0"/>
+    <origin xyz="0 0 0"/>
+    <inertia ixx="0" ixy="0" ixz="0" iyy="0" iyz="0" izz="0"/>
+  </inertial>
+</link>
+<joint name="stereo_camera_joint" type="fixed">
+  <parent link="base_link"/>
+  <child link="stereo_camera_link"/>
+  <origin xyz="0 -0.17589 0.05365" rpy="0 0 0"/>
+</joint>
+<link name="thermal_camera_link">
+  <visual>
+    <origin xyz="0 0 0" rpy="0 0 0"/>
+    <geometry>
+      <mesh filename="$(find rhex_description)/meshes/thermal_camera.stl" scale="1 1 1"/>
+    </geometry>
+    <material name="gray"/>
+  </visual>
+  <inertial>
+    <mass value="0"/>
+    <origin xyz="0 0 0"/>
+    <inertia ixx="0" ixy="0" ixz="0" iyy="0" iyz="0" izz="0"/>
+  </inertial>
+</link>
+<joint name="thermal_camera_joint" type="fixed">
+  <parent link="base_link"/>
+  <child link="thermal_camera_link"/>
+  <origin xyz="-0.00728 -0.18088 0.077" rpy="0 0 0"/>
+</joint>
+<link name="imu_link">
+  <visual>
+    <origin xyz="0 0 0" rpy="0 0 0"/>
+    <geometry>
+      <box size="0.01 0.01 0.002"/>
+    </geometry>
+    <material name="gray"/>
+  </visual>
+  <inertial>
+    <mass value="0"/>
+    <origin xyz="0 0 0"/>
+    <inertia ixx="0" ixy="0" ixz="0" iyy="0" iyz="0" izz="0"/>
+  </inertial>
+</link>
+<joint name="imu_joint" type="fixed">
+  <parent link="base_link"/>
+  <child link="imu_link"/>
+  <origin xyz="0 0 0.05" rpy="0 0 0"/>
+</joint>
   <gazebo reference="base_link">
     <self_collide>true</self_collide>
   </gazebo>
+<surface>
+  <friction>
+    <ode>
+      <mu>2.5</mu>
+      <mu2>2.5</mu2>
+    </ode>
+  </friction>
+  <contact>
+    <ode>
+      <kp>100000.0</kp>
+      <kd>10.0</kd>
+    </ode>
+  </contact>
+</surface>
   <!-- Legs -->
-  <xacro:leg_link name="front_left_leg" mesh="left_leg.stl"/>
-  <xacro:leg_link name="centre_left_leg" mesh="left_leg.stl"/>
-  <xacro:leg_link name="back_left_leg" mesh="left_leg.stl"/>
-  <xacro:leg_link name="front_right_leg" mesh="right_leg.stl"/>
-  <xacro:leg_link name="centre_right_leg" mesh="right_leg.stl"/>
-  <xacro:leg_link name="back_right_leg" mesh="right_leg.stl"/>
+  <xacro:leg_link name="front_left_leg" mesh="left_leg.stl" xyz="0.020502 0.028241 -0.039028"/>
+  <xacro:leg_link name="centre_left_leg" mesh="left_leg.stl" xyz="0.020502 0.028241 -0.039028"/>
+  <xacro:leg_link name="back_left_leg" mesh="left_leg.stl" xyz="0.020502 0.028241 -0.039028"/>
+  <xacro:leg_link name="front_right_leg" mesh="right_leg.stl" xyz="-0.020502 0.028241 -0.039028"/>
+  <xacro:leg_link name="centre_right_leg" mesh="right_leg.stl" xyz="-0.020502 0.028241 -0.039028"/>
+  <xacro:leg_link name="back_right_leg" mesh="right_leg.stl" xyz="-0.020502 0.028241 -0.039028"/>
   <!-- Leg joints -->
   <xacro:leg_joint name="front_left_leg_joint" parent="base_link" child="front_left_leg" xyz="0.11035 -0.135 0.04"/>
@@ -47,5 +137,3 @@
   <xacro:leg_joint name="back_right_leg_joint" parent="base_link" child="back_right_leg" xyz="-0.11035 0.135 0.04"/>
   <xacro:rhex_control/>
-  <!-- Sensors (inline for now) -->
-  <!-- LIDAR, cameras, IMU go here (copied from your current file) -->
 </robot>
